File: drivhus_pcb/drivhus_pcb.kicad_pcb (KiCad board)
At the start: 4 copper layers, 142.5 x 125 mm, 107 parts, among them J1 ESP32 pin side, J10 Sensor 6-10, J11 Temp/Humid/Light Indoors, J12 Temp/Humid Outdoors, J13 Pump 1-4, J14 Pump 5-8, J15 Pump 9-12, J16 Pump 13-15, J17 Waterlevel, J18 Growlight In, J19 -5V, J2 Water valve, J21 Fan, J22 Setup, J23 Growlight Out, J24 Growlight_-12V/-5V, J25 Waterpump_+12V/+5V, J26 Fan_-12V/-5V, J27 Fan_+12V/+5V, J28 Growlight_+12V/+5V, J3 ESP32 Power side, J33 Sensor 11-15, J34 Waterpump_-12V/-5V, J4 Sensor 1-5, J5 Conn_Coaxial_Power, J6 -12V, J7 12V Power connector, J8 +12V, J9 +5V, K16 Fan_relay, K17 Growlight_relay, K18 Watervalve_relay, Q1 30N06L-2, Q10 30N06L-11, Q11 30N06L-12, Q12 30N06L-13, Q13 30N06L-14, Q14 30N06L-15, Q15 30N06L-1, Q16 BC817, Q17 BC817, Q18 BC817, Q2 30N06L-3, Q3 30N06L-4, Q4 30N06L-5, Q5 30N06L-6, Q6 30N06L-7, Q7 30N06L-8, Q8 30N06L-9, Q9 30N06L-10, U1 CD74HC4067M, U2 CD74HC4067M

Commit message: Cannot use ADC2 together with WiFi on ESP32
Parts:
- added R38: 1K, Resistor_SMD:R_1206_3216Metric, F.Cu at (113.4, 87.9)
- added R39: 1.8K, Resistor_SMD:R_1206_3216Metric, F.Cu at (116.1, 87.9)
Connections:
- J3 pad 13: Net-(J3-Pin_13) -> Net-(J22-Pin_1)
- J3 pad 8: Net-(J22-Pin_1) -> Net-(J3-Pin_8)
- U1 pad 1: Net-(J3-Pin_13) -> Net-(U1-COM)
Routing:
- net Net-(U1-COM): track 0.00 -> 56.9 mm, vias 0 -> 2
- net Net-(J3-Pin_13): track 49.7 -> 0.00 mm, vias 1 -> 0
- net Net-(J22-Pin_1): track 5.93 -> 14.3 mm
- net Net-(J3-Pin_8): track 0.00 -> 6.52 mm
- net GND: vias 31 -> 32
Other:
- board text added: "1"
- board text added: "10"
- board text added: "11"
- board text added: "12"
- board text added: "13"
- board text added: "14"
- board text added: "15"
- board text added: "2"
- board text added: "3"
- board text added: "4"
- board text added: "5"
- board text added: "6"
- board text added: "7"
- board text added: "8"
- board text added: "9"
- board text added: "v7.1"
- board text removed: "v7.0"
